Commit message: Updated robot.xacro with camera_link and camera_joint
Fixed format

File: urdf/robot.xacro (robot description, xacro)
@@ -1,8 +1,9 @@
-<?xml version="1.0" ?>
+<?xml version="1.0"?>
 <robot name="robot" xmlns:xacro="http://www.ros.org/wiki/xacro">
     <xacro:include filename="$(find robot_description)/urdf/robot.gazebo" />
     <!-- Parameters -->
     <xacro:property name="chassis_mass" value="10" />
-    <xacro:property name="pi" value="3.1415926535897931"/>
+    <xacro:property name="pi" value="3.1415926535897931" />
+    <xacro:property name="camera_link" value="0.05" /> <!-- Size of square 'camera' box -->
     <!-- Link - chassis -->
     <link name="link_chassis">
@@ -44,5 +45,6 @@
             <mass value="1" />
             <origin xyz="0 0 0" rpy="0 0 0" />
-            <inertia ixx="0.002526666666667" ixy="0" ixz="0" iyy="0.002526666666667" iyz="0" izz="0.005"/>
+            <inertia ixx="0.002526666666667" ixy="0" ixz="0" iyy="0.002526666666667" iyz="0"
+                izz="0.005" />
         </inertial>
         <!-- Caster wheel support -->
@@ -93,5 +95,6 @@
             <mass value="1" />
             <origin xyz="0 0 0" rpy="0 0 0" />
-            <inertia ixx="0.002526666666667" ixy="0" ixz="0" iyy="0.002526666666667" iyz="0" izz="0.005"/>
+            <inertia ixx="0.002526666666667" ixy="0" ixz="0" iyy="0.002526666666667" iyz="0"
+                izz="0.005" />
         </inertial>
         <!-- Tires -->
@@ -99,5 +102,5 @@
             <origin rpy="${pi/2} 0 0" xyz="0 0.18 0" />
             <geometry>
-                <cylinder length="0.12" radius="0.4"/>
+                <cylinder length="0.12" radius="0.4" />
             </geometry>
         </collision>
@@ -115,5 +118,5 @@
             <origin rpy="${pi/2} 0 0" xyz="0 0.06 0" />
             <geometry>
-                <cylinder length="0.12" radius="0.08"/>
+                <cylinder length="0.12" radius="0.08" />
             </geometry>
         </collision>
@@ -121,5 +124,5 @@
             <origin rpy="${pi/2} 0 0" xyz="0 0.06 0" />
             <geometry>
-                <cylinder length="0.12" radius="0.08"/>
+                <cylinder length="0.12" radius="0.08" />
             </geometry>
             <material name="Grey">
@@ -152,5 +155,6 @@
             <mass value="1" />
             <origin xyz="0 0 0" rpy="0 0 0" />
-            <inertia ixx="0.002526666666667" ixy="0" ixz="0" iyy="0.002526666666667" iyz="0" izz="0.005"/>
+            <inertia ixx="0.002526666666667" ixy="0" ixz="0" iyy="0.002526666666667" iyz="0"
+                izz="0.005" />
         </inertial>
         <!-- Tires -->
@@ -158,5 +162,5 @@
             <origin rpy="${pi/2} 0 0" xyz="0 -0.18 0" />
             <geometry>
-                <cylinder length="0.12" radius="0.4"/>
+                <cylinder length="0.12" radius="0.4" />
             </geometry>
         </collision>
@@ -174,5 +178,5 @@
             <origin rpy="${pi/2} 0 0" xyz="0 -0.06 0" />
             <geometry>
-                <cylinder length="0.12" radius="0.08"/>
+                <cylinder length="0.12" radius="0.08" />
             </geometry>
         </collision>
@@ -180,5 +184,5 @@
             <origin rpy="${pi/2} 0 0" xyz="0 -0.06 0" />
             <geometry>
-                <cylinder length="0.12" radius="0.08"/>
+                <cylinder length="0.12" radius="0.08" />
             </geometry>
             <material name="Grey">
@@ -208,10 +212,11 @@
             <origin xyz="0 0 0" rpy="0 0 0" />
             <mass value="0.5" />
-            <inertia ixx="0.000252666666667" ixy="0" ixz="0" iyy="0.000252666666667" iyz="0" izz="0.0005"/>
-        </inertial>
-        <visual>
-            <origin xyz="0 0 0" rpy="0 0 0" />
-            <geometry>
-                <cylinder radius="0.15" length="0.20"/>
+            <inertia ixx="0.000252666666667" ixy="0" ixz="0" iyy="0.000252666666667" iyz="0"
+                izz="0.0005" />
+        </inertial>
+        <visual>
+            <origin xyz="0 0 0" rpy="0 0 0" />
+            <geometry>
+                <cylinder radius="0.15" length="0.20" />
             </geometry>
             <material name="Red">
@@ -220,9 +225,36 @@
         </visual>
         <collision>
-            <origin xyz="0 0 0" rpy="0 0 0"/>
-            <geometry>
-                <cylinder radius="0.15" length="0.20"/>
-            </geometry>
-        </collision>
+            <origin xyz="0 0 0" rpy="0 0 0" />
+            <geometry>
+                <cylinder radius="0.15" length="0.20" />
+            </geometry>
+        </collision>
+    </link>
+    <joint name="camera_joint" type="fixed">
+        <axis xyz="0 1 0" />
+        <origin xyz="${camera_link} 0 ${height3 - axel_offset*2}" rpy="0 0 0" />
+        <parent link="link3" />
+        <child link="camera_link" />
+    </joint>
+    <!-- Camera -->
+    <link name="camera_link">
+        <collision>
+            <origin xyz="0 0 0" rpy="0 0 0" />
+            <geometry>
+                <box size="${camera_link} ${camera_link} ${camera_link}" />
+            </geometry>
+        </collision>
+        <visual>
+            <origin xyz="0 0 0" rpy="0 0 0" />
+            <geometry>
+                <box size="${camera_link} ${camera_link} ${camera_link}" />
+            </geometry>
+            <material name="red" />
+        </visual>
+        <inertial>
+            <mass value="1e-5" />
+            <origin xyz="0 0 0" rpy="0 0 0" />
+            <inertia ixx="1e-6" ixy="0" ixz="0" iyy="1e-6" iyz="0" izz="1e-6" />
+        </inertial>
     </link>
     <!-- Robot tail -->
@@ -238,10 +270,11 @@
             <origin xyz="0 0 0" rpy="0 0 0" />
             <mass value="0.5" />
-            <inertia ixx="0.000252666666667" ixy="0" ixz="0" iyy="0.000252666666667" iyz="0" izz="0.0005"/>
+            <inertia ixx="0.000252666666667" ixy="0" ixz="0" iyy="0.000252666666667" iyz="0"
+                izz="0.0005" />
         </inertial>
         <visual>
             <origin xyz="-0.2 0 0" rpy="0 ${pi/2} 0" />
             <geometry>
-                <cylinder radius="0.05" length="0.40"/>
+                <cylinder radius="0.05" length="0.40" />
             </geometry>
             <material name="Red">
@@ -250,7 +283,7 @@
         </visual>
         <collision>
-            <origin xyz="-0.2 0 0" rpy="0 ${pi/2} 0"/>
-            <geometry>
-                <cylinder radius="0.05" length="0.40"/>
+            <origin xyz="-0.2 0 0" rpy="0 ${pi/2} 0" />
+            <geometry>
+                <cylinder radius="0.05" length="0.40" />
             </geometry>
         </collision>

Commit message: Updated camera_joint origin and parent link

File: urdf/robot.xacro (robot description, xacro)
@@ -233,6 +233,6 @@
     <joint name="camera_joint" type="fixed">
         <axis xyz="0 1 0" />
-        <origin xyz="${camera_link} 0 ${height3 - axel_offset*2}" rpy="0 0 0" />
-        <parent link="link3" />
+        <origin xyz="1 0 0" rpy="0 0 0" />
+        <parent link="link_chassis" />
         <child link="camera_link" />
     </joint>

Commit message: Updated material colors in robot.xacro

File: urdf/robot.xacro (robot description, xacro)
@@ -221,5 +221,5 @@
             </geometry>
             <material name="Red">
-                <color rgba="0.7 0.1 0.1 1" />
+                <color rgba="1 0 0 1" />
             </material>
         </visual>
@@ -250,5 +250,5 @@
                 <box size="${camera_link} ${camera_link} ${camera_link}" />
             </geometry>
-            <material name="red" />
+            <material name="Red" />
         </visual>
         <inertial>
@@ -279,5 +279,5 @@
             </geometry>
             <material name="Red">
-                <color rgba="0.7 0.1 0.1 1" />
+                <color rgba="1 0 0 1" />
             </material>
         </visual>
